File: PCB-Files/esp32/beta/top/top.sch (EAGLE design)
At the start: 5 parts

Commit message: creates final PCB version; revised beta side pcbs to match beta main pcb pinouts
Parts:
- removed HALL_1_IN, HALL_GND, HALL_VCC: TPTP20SQ, testpad:TPTP20SQ
- added TP1, TP10, TP11, TP12, TP13, TP14, TP15, TP16, TP17, TP18, TP19, TP2, TP3, TP4, TP5, TP6, TP7, TP8, TP9: TPTP10SQ, testpad:TPTP10SQ
Connections:
- new net HALL_2: HALL.SIG, TP3.TP, TP7.TP
- new net TOUCH: TP15.TP, TP16.TP, TP17.TP, TP18.TP, TP19.TP
- net GND: now also TP12.TP, TP14.TP, TP4.TP, TP8.TP; no longer HALL_GND.TP
- net HALL_1: now also TP10.TP, TP13.TP, TP2.TP, TP6.TP; no longer HALL.SIG, HALL_1_IN.TP
- net VCC: now also TP1.TP, TP11.TP, TP5.TP, TP9.TP; no longer HALL_VCC.TP
